File: NeoPixel_2026_Robot.kicad_pcb (KiCad board)
At the start: 2 copper layers, 31 parts, among them J1 Pixcel1, J10 XT30, J2 Pixcel2, J3 Pixcel3, J4 Pixcel4, J5 INPUT, J6 EM-IN1, J7 EM-IN2, J8 EM-IN3, J9 EM-IN4, U1 TLP291, U2 TLP291, U3 TLP291, U4 TLP291

Commit message: おためし
Parts:
- moved H3 83.0 mm to (91.4, 68.0)
- moved JP4 83.0 mm to (120.3, 82.7)
- moved A1 83.0 mm to (69.8, 51.2)
- moved H1 83.0 mm to (91.4, 50.9)
- moved H2 83.0 mm to (91.4, 59.5)
- moved H4 83.0 mm to (91.4, 76.6)
- moved J1 83.0 mm to (117.3, 70.9)
- moved J2 83.0 mm to (100.0, 50.9)
- moved J3 83.0 mm to (100.0, 59.5)
- moved J4 83.0 mm to (100.0, 68.0)
- moved J5 83.0 mm to (107.8, 92.0)
- moved J6 83.0 mm to (107.8, 50.9)
- moved J7 83.0 mm to (107.8, 59.3)
- moved J8 83.0 mm to (107.8, 67.8)
- moved J9 83.0 mm to (107.8, 76.2)
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
Commit message: windowsのほうで作ってたところまで手動復元
Parts:
- added J11: Type-C, NeoPixcel_2026_Robot_Lib:PowerOnlyUSB_C, F.Cu at (54.5, 22.4)
- J2, J3, J4: footprint MountingHole:MountingHole_3.5mm_Pad -> Connector_JST:JST_XA_B03B-XASK-1_1x03_P2.50mm_Vertical
- moved J1 101.5 mm to (40.9, 4.16)
- moved J5 89.6 mm to (31.3, 45.3)
- moved J6 89.6 mm to (31.3, 4.16)
- moved J7 89.6 mm to (31.3, 12.6)
- moved J8 89.6 mm to (31.3, 21.1)
- moved J9 89.6 mm to (31.3, 29.5)
- moved JP2 89.6 mm to (34.7, 36.0)
- moved JP3 89.6 mm to (39.2, 36.0)
- moved JP4 89.6 mm to (43.8, 36.0)
- moved JP1 89.6 mm to (30.1, 36.0)
- moved H1 82.4 mm to (23.5, 4.21)
- moved H2 82.4 mm to (23.5, 12.8)
- moved H3 82.4 mm to (23.5, 21.3)
- moved H4 82.4 mm to (23.5, 29.9)
- moved A1 82.4 mm to (1.95, 4.52)
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
Commit message: ライブラリをグローバルからプロジェクト専用のものに変更した
Parts:
- removed J11: Type-C, NeoPixcel_2026_Robot_Lib:PowerOnlyUSB_C
- moved U1 38.9 mm to (39.0, 35.6)
- moved U2 38.9 mm to (39.0, 39.8)
- moved U3 38.9 mm to (39.0, 43.9)
- moved U4 38.9 mm to (39.0, 48.0)
- moved J5 28.8 mm to (3.02, 51.0)
- moved J10 27.0 mm to (29.0, 47.6)
- moved JP1 17.6 mm to (36.5, 52.4)
- moved JP2 17.6 mm to (41.1, 52.4)
- moved JP3 17.6 mm to (45.7, 52.4)
- moved JP4 17.6 mm to (50.2, 52.4)
- moved J4 0.73 mm to (40.5, 28.9)
- moved J9 0.73 mm to (30.9, 28.9)
- moved J1 0.73 mm to (40.5, 3.55)
- moved J2 0.73 mm to (40.5, 12.0)
- moved J3 0.73 mm to (40.5, 20.4)
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
Commit message: 作業を進めた 非常に迷走中
Parts:
- added J11: Type-C, ProjectLib:PowerOnlyUSB_C, F.Cu at (53.5, 21.4)
- R1, R2, R3, R4, R5, R6, R7, R8, U1, U2, U3, U4: moved to B.Cu
- moved H3 166.0 mm to (171.0, 96.0)
- moved A1 156.8 mm to (149.4, 56.1)
- moved H4 150.0 mm to (171.0, 54.0)
- moved H2 116.5 mm to (104.0, 96.0)
- moved J5 109.6 mm to (109.3, 78.0), turned to -90 degrees
- moved R2 97.0 mm to (119.5, 71.9), turned to 180 degrees
- moved H1 95.3 mm to (104.0, 54.0)
- moved R4 90.8 mm to (119.5, 67.9), turned to 180 degrees
- moved R1 90.6 mm to (107.0, 71.9)
- moved R6 85.1 mm to (119.5, 63.9), turned to 180 degrees
- moved R3 83.7 mm to (107.0, 67.9)
- moved U1 82.4 mm to (113.2, 71.2)
- moved R8 80.1 mm to (119.5, 59.9), turned to 180 degrees
- moved U2 79.2 mm to (113.2, 67.2)
- moved R5 77.2 mm to (107.0, 63.9)
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Connections:
- A1 pad 10: /Pixcel1 -> /Pixcel2
- A1 pad 11: /Pixcel2 -> /Pixcel3
- A1 pad 12: /Pixcel3 -> /Pixcel4
- A1 pad 13: /Pixcel4 -> /EM-sig
- A1 pad 5: /Sig1_OUT -> /Sig4_OUT
- A1 pad 6: /Sig2_OUT -> /Sig3_OUT
- A1 pad 7: /Sig3_OUT -> /Sig2_OUT
- A1 pad 8: /Sig4_OUT -> /Sig1_OUT
- A1 pad 9: /EM-sig -> /Pixcel1
- R6 pad 1: /Sig4_IN -> +5V
- R6 pad 2: Net-(R6-Pad2) -> /Sig3_OUT
- R7 pad 1: +5V -> /Sig4_IN
- R7 pad 2: /Sig3_OUT -> Net-(R7-Pad2)
- U4 pad 1: Net-(R6-Pad2) -> Net-(R7-Pad2)
Routing:
- net /Sig1_OUT: track 0.00 -> 26.7 mm
- net /Sig2_OUT: track 0.00 -> 25.2 mm
- net /Sig3_OUT: track 0.00 -> 23.1 mm
- net /Sig4_OUT: track 0.00 -> 21.4 mm
- net Net-(R7-Pad2): track 0.00 -> 2.09 mm
- net Net-(R5-Pad2): track 0.00 -> 2.09 mm
- net Net-(R3-Pad2): track 0.00 -> 2.09 mm
- net Net-(R1-Pad2): track 0.00 -> 2.09 mm
Other:
- board outline added: 75 x 50 mm

Commit message: ちょっとずつ進んでいる フォトかプラのプルアップ抵抗をスルーホールにしたほうがええかもしれない
Parts:
- moved R1 2.29 mm to (104.7, 71.9)
- moved R2 2.29 mm to (117.2, 71.9)
- moved R3 2.29 mm to (104.7, 67.9)
- moved R4 2.29 mm to (117.2, 67.9)
- moved R5 2.29 mm to (104.7, 63.9)
- moved R6 2.29 mm to (117.2, 63.9)
- moved R7 2.29 mm to (104.7, 59.9)
- moved R8 2.29 mm to (117.2, 59.9)
- moved U1 2.29 mm to (111.0, 71.2)
- moved U2 2.29 mm to (111.0, 67.2)
- moved U3 2.29 mm to (111.0, 63.2)
- moved U4 2.29 mm to (111.0, 59.2)
Connections:
- A1 pad 5: /Sig4_OUT -> /Sig1_OUT
- A1 pad 6: /Sig3_OUT -> /Sig2_OUT
- A1 pad 7: /Sig2_OUT -> /Sig3_OUT
- A1 pad 8: /Sig1_OUT -> /Sig4_OUT
Routing:
- net /Sig4_IN: track 0.00 -> 30.4 mm
- net /Sig1_OUT: track 26.7 -> 2.09 mm
- net /Sig3_IN: track 0.00 -> 23.1 mm
- net /Sig2_OUT: track 25.2 -> 2.45 mm
- net /Sig3_OUT: track 23.1 -> 2.45 mm
- net /Sig4_OUT: track 21.4 -> 2.45 mm
- net /Sig2_IN: track 0.00 -> 15.7 mm
- net +5V: track 0.00 -> 12.0 mm
- net /Sig1_IN: track 0.00 -> 8.39 mm
- added copper zone on B.Cu, net GND

Commit message: スルーホールにしたが、締まらない
Parts:
- removed R2, R4, R6, R8: R, Resistor_SMD:R_0603_1608Metric_Pad0.98x0.95mm_HandSolder
- moved J1 143.0 mm to (138.8, 70.8)
- moved J2 143.0 mm to (138.8, 79.3)
- moved J3 143.0 mm to (138.8, 87.8)
- moved J4 143.0 mm to (138.8, 96.2)
- moved J6 143.0 mm to (129.2, 70.8)
- moved J7 143.0 mm to (129.2, 79.3)
- moved J8 143.0 mm to (129.2, 87.8)
- moved J9 143.0 mm to (129.2, 96.2)
Routing:
- net +5V: track 12.0 -> 0.00 mm
- net Net-(R7-Pad2): track 2.09 -> 0.00 mm

Commit message: 色々変更した 具体的なところは覚えていない
Parts:
- added R2: R, Resistor_THT:R_Axial_DIN0207_L6.3mm_D2.5mm_P10.16mm_Horizontal, F.Cu at (50.6, 18.2)
- added R4: R, Resistor_THT:R_Axial_DIN0207_L6.3mm_D2.5mm_P10.16mm_Horizontal, F.Cu at (50.6, 22.3)
- added R6: R, Resistor_THT:R_Axial_DIN0207_L6.3mm_D2.5mm_P10.16mm_Horizontal, F.Cu at (50.6, 26.3)
- added R8: R, Resistor_THT:R_Axial_DIN0207_L6.3mm_D2.5mm_P10.16mm_Horizontal, F.Cu at (50.6, 30.4)
- R1, R3, R5, R7, U1, U2, U3, U4: moved to F.Cu
- moved H3 165.8 mm to (23.2, 21.0)
- moved A1 156.6 mm to (1.63, 4.20)
- moved H4 149.8 mm to (23.2, 29.5)
- moved J3 118.9 mm to (40.5, 20.7)
- moved J4 118.9 mm to (40.5, 29.2)
- moved J6 118.9 mm to (31.0, 3.84)
- moved J7 118.9 mm to (31.0, 12.3)
- moved J8 118.9 mm to (31.0, 20.7)
- moved J9 118.9 mm to (31.0, 29.2)
- moved J1 118.9 mm to (40.5, 3.84)
- moved J2 118.9 mm to (40.5, 12.3)
- moved H2 116.2 mm to (23.2, 12.4)
- moved H1 95.1 mm to (23.2, 3.89)
- moved R1 92.2 mm to (15.6, 48.1)
- moved R3 90.7 mm to (15.6, 50.6)
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Routing:
- net /Sig4_IN: track 30.4 -> 0.00 mm
- net /Sig3_IN: track 23.1 -> 0.00 mm
- net /Sig2_IN: track 15.7 -> 0.00 mm
- net /Sig1_IN: track 8.39 -> 0.00 mm
- net /Sig4_OUT: track 2.45 -> 0.00 mm
- net /Sig3_OUT: track 2.45 -> 0.00 mm
- net /Sig2_OUT: track 2.45 -> 0.00 mm
- net Net-(R5-Pad2): track 2.09 -> 0.00 mm
- net Net-(R3-Pad2): track 2.09 -> 0.00 mm
- net Net-(R1-Pad2): track 2.09 -> 0.00 mm
- net /Sig1_OUT: track 2.09 -> 0.00 mm
- removed copper zone on B.Cu, net GND
Other:
- board outline removed
